File: corneds_devkit/io_board/io.kicad_sch (KiCad schematic)
At the start: 0 parts

Commit message: finished schematic for io board
Parts:
- added J1, J2, J3, J4: Conn_01x14_Female, symbol Connector:Conn_01x14_Female
Connections:
- new net GNDL: J1.14 (Pin_14)
- new net GNDR: J4.14 (Pin_14)
- new net VDDL: J1.1 (Pin_1)
- new net VDDR: J4.1 (Pin_1)
- new net VJOYL: J2.1 (Pin_1)
- new net VJOYR: J3.1 (Pin_1)
- new net key_a: J1.10 (Pin_10)
- new net key_alt: J3.11 (Pin_11)
- new net key_apos: J4.9 (Pin_9)
- new net key_b: J2.10 (Pin_10)
- new net key_bslash: J3.6 (Pin_6)
- new net key_c: J2.8 (Pin_8)
- new net key_comma: J3.8 (Pin_8)
- new net key_ctrl: J1.9 (Pin_9)
- new net key_d: J1.12 (Pin_12)
- new net key_del: J4.3 (Pin_3)
- new net key_e: J1.6 (Pin_6)
- new net key_enter: J3.13 (Pin_13)
- new net key_esc: J1.3 (Pin_3)
- new net key_f: J1.13 (Pin_13)
- new net key_g: J2.4 (Pin_4)
- new net key_h: J3.4 (Pin_4)
- new net key_i: J4.6 (Pin_6)
- new net key_j: J4.13 (Pin_13)
- new net key_k: J4.12 (Pin_12)
- new net key_l: J4.11 (Pin_11)
- new net key_lclick: J2.14 (Pin_14)
- new net key_lower: J3.12 (Pin_12)
- new net key_lshift: J2.5 (Pin_5)
- new net key_m: J3.9 (Pin_9)
- new net key_mod: J2.11 (Pin_11)
- new net key_n: J3.10 (Pin_10)
- new net key_o: J4.5 (Pin_5)
- new net key_p: J4.4 (Pin_4)
- new net key_period: J3.7 (Pin_7)
- new net key_q: J1.4 (Pin_4)
- new net key_r: J1.7 (Pin_7)
- new net key_raise: J2.12 (Pin_12)
- new net key_rclick: J3.14 (Pin_14)
- new net key_rshift: J3.5 (Pin_5)
- new net key_s: J1.11 (Pin_11)
- new net key_semi: J4.10 (Pin_10)
- new net key_space: J2.13 (Pin_13)
- new net key_t: J1.8 (Pin_8)
- new net key_u: J4.7 (Pin_7)
- new net key_v: J2.9 (Pin_9)
- new net key_w: J1.5 (Pin_5)
- new net key_x: J2.7 (Pin_7)
- new net key_y: J4.8 (Pin_8)
- new net key_z: J2.6 (Pin_6)
- new net left_led_di: J1.2 (Pin_2)
- new net mouse_x: J3.2 (Pin_2)
- new net mouse_y: J3.3 (Pin_3)
- new net right_led_di: J4.2 (Pin_2)
- new net scroll_x: J2.2 (Pin_2)
- new net scroll_y: J2.3 (Pin_3)
