File: corneds_devkit/io_board/io.kicad_sch (KiCad schematic)
At the start: 10 parts, among them J1 Conn_01x09_Pin, J2 JOY_VSEL

Commit message: replaced io board headers with 2.54mm and added pullups to i2c lines
Parts:
- J1: footprint Connector_PinHeader_1.27mm:PinHeader_1x09_P1.27mm_Vertical -> Connector_PinSocket_2.54mm:PinSocket_1x09_P2.54mm_Vertical
- J2: footprint Connector_PinHeader_1.27mm:PinHeader_1x03_P1.27mm_Vertical -> Connector_PinSocket_2.54mm:PinSocket_1x03_P2.54mm_Vertical
