File: corneds_devkit/io_board/right_mouse.kicad_sch (KiCad schematic)
At the start: 0 parts

Commit message: finished mouse and key boards
Parts:
- added D87: APA-106-F5, LED_THT:LED_D5.0mm-4_RGB, symbol LED:APA-106-F5
- added D88: 1N4148W, Diode_SMD:D_SOD-123, symbol Diode:1N4148W
- added SW44: SW_Push, symbol Switch:SW_Push
- added U2: COM-09426, symbol entropy:COM-09426
Connections:
- new net: D88.2 (A), SW44.2
- new net GNDL: D87.2 (GND), U2.4 (GND)
- new net VDDR: D87.3 (VDD), SW44.1
- new net VJOYR: U2.2 (VDD)
- new net key_rclick: D88.1 (K)
- new net mouse_x: U2.1 (x-axis)
- new net mouse_y: U2.3 (y-axis)
- new net rclick_led_di: D87.4 (DI)

Commit message: finished schematic for io board
Connections:
- net GNDL renamed GNDR
Changed lines of the file:
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@@
+		)
+	)
+	(global_label "GNDR"
+		(shape input)
+		(at 163.83 101.6 270)
+		(fields_autoplaced yes)
+		(effects
+			(font
+				(size 1.27 1.27)
+			)
+			(justify right)
+		)
+		(property "Intersheetrefs" "${INTERSHEET_REFS}"
+			(at 163.83 109.7257 90)
+			(effects
+				(font
+					(size 1.27 1.27)
+				)
+				(justify right)
+				(hide yes)
+			)
+		)
+	)
+	(global_label "VJOYR"
+		(shape input)
+		(at 114.3 71.12 90)
+		(fields_autoplaced yes)
+		(effects
+			(font
+				(size 1.27 1.27)
+			)
+			(justify left)
+		)
+		(property "Intersheetrefs" "${INTERSHEET_REFS}"
+			(at 114.3 62.3895 90)
+			(effects
+				(font
+					(size 1.27 1.27)
+				)
+				(justify left)
+				(hide yes)
+			)
+		)
+	)
+	(global_label "VDDR"
+		(shape input)
+		(at 154.94 71.12 90)
+		(fields_autoplaced yes)
+		(effects
+			(font
+				(size 1.27 1.27)
+			)
+			(justify left)
+		)
+		(property "Intersheetrefs" "${INTERSHEET_REFS}"
+			(at 154.94 63.2362 90)
+			(effects
+				(font
+					(size 1.27 1.27)
+				)
+				(justify left)
+				(hide yes)
+			)
 		)
 	)
@@
 					(unit 1)
 				)
-			)
-		)
-	)
-	(symbol
-		(lib_id "power:GND")
-		(at 163.83 101.6 0)
-		(unit 1)
-		(exclude_from_sim no)
-		(in_bom yes)
-		(on_board yes)
-		(dnp no)
-		(fields_autoplaced yes)
-		(property "Reference" "#PWR010"
-			(at 163.83 107.95 0)
-			(effects
-				(font
-					(size 1.27 1.27)
-				)
-				(hide yes)
-			)
-		)
-		(property "Value" "GNDL"
-			(at 163.83 106.68 0)
-			(effects
-				(font
-					(size 1.27 1.27)
-				)
-			)
-		)
-		(property "Footprint" ""
-			(at 163.83 101.6 0)
-			(effects
-				(font
-					(size 1.27 1.27)
-				)
-				(hide yes)
-			)
-		)
-		(property "Datasheet" ""
-			(at 163.83 101.6 0)
-			(effects
-				(font
-					(size 1.27 1.27)
-				)
-				(hide yes)
-			)
-		)
-		(property "Description" "Power symbol creates a global label with name \"GND\" , ground"
-			(at 163.83 101.6 0)
-			(effects
-				(font
-					(size 1.27 1.27)
-				)
-				(hide yes)
-			)
-		)
-		(pin "1"
-		)
-		(instances
-			(project "io_board"
-				(path "/244b6d6b-132d-4d50-ae86-e41103b29008/d0a6750f-d35a-4f18-ad73-a13ad9a077bd"
-					(reference "#PWR010")
-					(unit 1)
-				)
-			)
-		)
-	)
-	(symbol
-		(lib_id "power:VDD")
-		(at 114.3 71.12 0)
-		(unit 1)
-		(exclude_from_sim no)
-		(in_bom yes)
-		(on_board yes)
-		(dnp no)
-		(fields_autoplaced yes)
-		(property "Reference" "#PWR08"
-			(at 114.3 74.93 0)
-			(effects
-				(font
-					(size 1.27 1.27)
-				)
-				(hide yes)
-			)
-		)
-		(property "Value" "VJOYR"
-			(at 114.3 66.04 0)
-			(effects
-				(font
-					(size 1.27 1.27)
-				)
-			)
-		)
-		(property "Footprint" ""
-			(at 114.3 71.12 0)
-			(effects
-				(font
-					(size 1.27 1.27)
-				)
-				(hide yes)
-			)
-		)
-		(property "Datasheet" ""
-			(at 114.3 71.12 0)
-			(effects
-				(font
-					(size 1.27 1.27)
-				)
-				(hide yes)
-			)
-		)
-		(property "Description" "Power symbol creates a global label with name \"VDD\""
-			(at 114.3 71.12 0)
-			(effects
-				(font
-					(size 1.27 1.27)
-				)
-				(hide yes)
-			)
-		)
-		(pin "1"
-		)
-		(instances
-			(project "io_board"
-				(path "/244b6d6b-132d-4d50-ae86-e41103b29008/d0a6750f-d35a-4f18-ad73-a13ad9a077bd"
-					(reference "#PWR08")
-					(unit 1)
-				)
-			)
-		)
-	)
-	(symbol
-		(lib_id "power:VDD")
-		(at 154.94 71.12 0)
-		(unit 1)
-		(exclude_from_sim no)
-		(in_bom yes)
-		(on_board yes)
-		(dnp no)
-		(fields_autoplaced yes)
-		(property "Reference" "#PWR09"
-			(at 154.94 74.93 0)
-			(effects
-				(font
-					(size 1.27 1.27)
-				)
-				(hide yes)
-			)
-		)
-		(property "Value" "VDDR"
-			(at 154.94 66.04 0)
-			(effects
-				(font
-					(size 1.27 1.27)
-				)
-			)
-		)
-		(property "Footprint" ""
-			(at 154.94 71.12 0)
-			(effects
-				(font
-					(size 1.27 1.27)
-				)
-				(hide yes)
-			)
-		)
-		(property "Datasheet" ""
-			(at 154.94 71.12 0)
-			(effects
-				(font
-					(size 1.27 1.27)
-				)
-				(hide yes)
-			)
-		)
-		(property "Description" "Power symbol creates a global label with name \"VDD\""
-			(at 154.94 71.12 0)
-			(effects
-				(font
-					(size 1.27 1.27)
-				)
-				(hide yes)
-			)
-		)
-		(pin "1"
-		)
-		(instances
-			(project "io_board"
-				(path "/244b6d6b-132d-4d50-ae86-e41103b29008/d0a6750f-d35a-4f18-ad73-a13ad9a077bd"
-					(reference "#PWR09")
-					(unit 1)
-				)

Commit message: re-routed io board with keypad IC
Parts:
- removed D88: 1N4148W, Diode_SMD:D_SOD-123, symbol Diode:1N4148W
Connections:
- net VDDR: no longer SW44.1
- net ROW3R: now reaches SW44.2
- new net COL2R: SW44.1
Changed lines of the file:
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@@
 	(paper "A4")
-	(junction
-		(at 154.94 81.28)
-		(diameter 0)
-		(color 0 0 0 0)
-	)
 	(junction
 		(at 163.83 100.33)
@@
 	(wire
 		(pts
+			(xy 154.94 81.28) (xy 154.94 76.2)
+		)
+		(stroke
+			(width 0)
+			(type default)
+		)
+	)
+	(wire
+		(pts
+			(xy 114.3 71.12) (xy 114.3 76.2)
+		)
+		(stroke
+			(width 0)
+			(type default)
+		)
+	)
+	(wire
+		(pts
+			(xy 125.73 86.36) (xy 128.27 86.36)
+		)
+		(stroke
+			(width 0)
+			(type default)
+		)
+	)
+	(wire
+		(pts
 			(xy 158.75 81.28) (xy 154.94 81.28)
 		)
@@
 	(wire
 		(pts
-			(xy 114.3 71.12) (xy 114.3 76.2)
-		)
-		(stroke
-			(width 0)
-			(type default)
-		)
-	)
-	(wire
-		(pts
-			(xy 125.73 86.36) (xy 128.27 86.36)
-		)
-		(stroke
-			(width 0)
-			(type default)
-		)
-	)
-	(wire
-		(pts
-			(xy 177.8 81.28) (xy 180.34 81.28)
-		)
-		(stroke
-			(width 0)
-			(type default)
-		)
-	)
-	(wire
-		(pts
 			(xy 163.83 100.33) (xy 163.83 101.6)
 		)
@@
 	(wire
 		(pts
+			(xy 168.91 81.28) (xy 172.72 81.28)
+		)
+		(stroke
+			(width 0)
+			(type default)
+		)
+	)
+	(wire
+		(pts
 			(xy 125.73 81.28) (xy 128.27 81.28)
 		)
@@
 	(wire
 		(pts
-			(xy 154.94 81.28) (xy 154.94 85.09)
-		)
-		(stroke
-			(width 0)
-			(type default)
-		)
-	)
-	(wire
-		(pts
-			(xy 154.94 71.12) (xy 154.94 81.28)
+			(xy 144.78 80.01) (xy 144.78 85.09)
 		)
 		(stroke
@@
 	(wire
 		(pts
-			(xy 163.83 85.09) (xy 154.94 85.09)
+			(xy 163.83 85.09) (xy 144.78 85.09)
 		)
 		(stroke
@@
 		)
 	)
-	(wire
-		(pts
-			(xy 168.91 81.28) (xy 170.18 81.28)
-		)
-		(stroke
-			(width 0)
-			(type default)
+	(global_label "COL2R"
+		(shape input)
+		(at 154.94 76.2 90)
+		(fields_autoplaced yes)
+		(effects
+			(font
+				(size 1.27 1.27)
+			)
+			(justify left)
+		)
+		(property "Intersheetrefs" "${INTERSHEET_REFS}"
+			(at 154.94 67.1067 90)
+			(effects
+				(font
+					(size 1.27 1.27)
+				)
+				(justify left)
+				(hide yes)
+			)
 		)
 	)
@@
 		)
 	)
+	(global_label "ROW3R"
+		(shape input)
+		(at 172.72 81.28 0)
+		(fields_autoplaced yes)
+		(effects
+			(font
+				(size 1.27 1.27)
+			)
+			(justify left)
+		)
+		(property "Intersheetrefs" "${INTERSHEET_REFS}"
+			(at 182.2366 81.28 0)
+			(effects
+				(font
+					(size 1.27 1.27)
+				)
+				(justify left)
+				(hide yes)
+			)
+		)
+	)
 	(global_label "GNDR"
 		(shape input)
@@
 	(global_label "VDDR"
 		(shape input)
-		(at 154.94 71.12 90)
-		(fields_autoplaced yes)
-		(effects
-			(font
-				(size 1.27 1.27)
-			)
-			(justify left)
-		)
-		(property "Intersheetrefs" "${INTERSHEET_REFS}"
-			(at 154.94 63.2362 90)
-			(effects
-				(font
-					(size 1.27 1.27)
-				)
-				(justify left)
-				(hide yes)
-			)
-		)
-	)
-	(global_label "key_rclick"
-		(shape input)
-		(at 180.34 81.28 0)
-		(fields_autoplaced yes)
-		(effects
-			(font
-				(size 1.27 1.27)
-			)
-			(justify left)
-		)
-		(property "Intersheetrefs" "${INTERSHEET_REFS}"
-			(at 192.6386 81.28 0)
+		(at 144.78 80.01 90)
+		(fields_autoplaced yes)
+		(effects
+			(font
+				(size 1.27 1.27)
+			)
+			(justify left)
+		)
+		(property "Intersheetrefs" "${INTERSHEET_REFS}"
+			(at 144.78 72.1262 90)
 			(effects
 				(font
@@
 			)
 		)
-	)
-	(symbol
-		(lib_id "Diode:1N4148W")
-		(at 173.99 81.28 180)
-		(unit 1)
-		(exclude_from_sim no)
-		(in_bom yes)
-		(on_board yes)
-		(dnp no)
-		(fields_autoplaced yes)
-		(property "Reference" "D88"
-			(at 173.99 74.93 0)
-			(effects
-				(font
-					(size 1.27 1.27)
-				)
-			)
-		)
-		(property "Value" "1N4148W"
-			(at 173.99 77.47 0)
-			(effects
-				(font
-					(size 1.27 1.27)
-				)
-			)
-		)
-		(property "Footprint" "Diode_SMD:D_SOD-123"
-			(at 173.99 76.835 0)
-			(effects
-				(font
-					(size 1.27 1.27)
-				)
-				(hide yes)
-			)
-		)
-		(property "Datasheet" "https://www.vishay.com/docs/85748/1n4148w.pdf"
-			(at 173.99 81.28 0)
-			(effects
-				(font
-					(size 1.27 1.27)
-				)
-				(hide yes)
-			)
-		)
-		(property "Description" "75V 0.15A Fast Switching Diode, SOD-123"
-			(at 173.99 81.28 0)
-			(effects
-				(font
-					(size 1.27 1.27)
-				)
-				(hide yes)
-			)
-		)
-		(pin "1"
-		)
-		(pin "2"
-		)
-		(instances
-			(project "io_board"
-				(path "/244b6d6b-132d-4d50-ae86-e41103b29008/d0a6750f-d35a-4f18-ad73-a13ad9a077bd"
-					(reference "D88")
-					(unit 1)
-				)
-			)
-		)

Commit message: added switch footprint, io sch, and keypad IC footprint. Need to find new LEDs and make joystick footprint
Parts:
- SW44: footprint (none) -> key-switches:SW_Gateron_LowProfile_HotSwap_THT
Connections:
- net VDDR renamed VDD_3V3R
Changed lines of the file:
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@@
 		)
 	)
-	(global_label "VDDR"
+	(global_label "VDD_3V3R"
 		(shape input)
 		(at 144.78 80.01 90)
@@
 		)
 		(property "Intersheetrefs" "${INTERSHEET_REFS}"
-			(at 144.78 72.1262 90)
+			(at 144.78 67.651 90)
 			(effects
 				(font
@@
 			)
 		)
-		(property "Footprint" ""
+		(property "Footprint" "key-switches:SW_Gateron_LowProfile_HotSwap_THT"
 			(at 163.83 76.2 0)
 			(effects

Commit message: io sch done. Need to route
Parts:
- D87: value APA-106-F5 -> SK68XX-SIDE; footprint LED_THT:LED_D5.0mm-4_RGB -> entropy:SK68XX-SIDE
- U2: footprint (none) -> entropy:COM-09426
Connections:
- net VDD_3V3R renamed VDD_5VR
Other:
- moved on the sheet: U2
Changed lines of the file:
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@@
 	(wire
 		(pts
-			(xy 125.73 86.36) (xy 128.27 86.36)
+			(xy 127 86.36) (xy 130.81 86.36)
 		)
 		(stroke
@@
 	(wire
 		(pts
-			(xy 125.73 81.28) (xy 128.27 81.28)
+			(xy 127 81.28) (xy 130.81 81.28)
 		)
 		(stroke
@@
 	(global_label "mouse_y"
 		(shape input)
-		(at 128.27 86.36 0)
-		(fields_autoplaced yes)
-		(effects
-			(font
-				(size 1.27 1.27)
-			)
-			(justify left)
-		)
-		(property "Intersheetrefs" "${INTERSHEET_REFS}"
-			(at 139.2984 86.36 0)
+		(at 130.81 86.36 0)
+		(fields_autoplaced yes)
+		(effects
+			(font
+				(size 1.27 1.27)
+			)
+			(justify left)
+		)
+		(property "Intersheetrefs" "${INTERSHEET_REFS}"
+			(at 141.8384 86.36 0)
 			(effects
 				(font
@@
 		)
 	)
-	(global_label "VDD_3V3R"
+	(global_label "VDD_5VR"
 		(shape input)
 		(at 144.78 80.01 90)
@@
 		)
 		(property "Intersheetrefs" "${INTERSHEET_REFS}"
-			(at 144.78 67.651 90)
+			(at 144.78 68.8605 90)
 			(effects
 				(font
@@
 	(global_label "mouse_x"
 		(shape input)
-		(at 128.27 81.28 0)
-		(fields_autoplaced yes)
-		(effects
-			(font
-				(size 1.27 1.27)
-			)
-			(justify left)
-		)
-		(property "Intersheetrefs" "${INTERSHEET_REFS}"
-			(at 139.3589 81.28 0)
+		(at 130.81 81.28 0)
+		(fields_autoplaced yes)
+		(effects
+			(font
+				(size 1.27 1.27)
+			)
+			(justify left)
+		)
+		(property "Intersheetrefs" "${INTERSHEET_REFS}"
+			(at 141.8989 81.28 0)
 			(effects
 				(font
@@
 			)
 		)
-		(property "Value" "APA-106-F5"
+		(property "Value" "SK68XX-SIDE"
 			(at 176.53 86.3914 0)
 			(effects
@@
 			)
 		)
-		(property "Footprint" "LED_THT:LED_D5.0mm-4_RGB"
+		(property "Footprint" "entropy:SK68XX-SIDE"
 			(at 165.1 100.33 0)
 			(effects
@@
 			)
 		)
-		(property "Datasheet" "https://cdn.sparkfun.com/datasheets/Components/LED/COM-12877.pdf"
+		(property "Datasheet" "https://www.digikey.com/en/products/detail/adafruit-industries-llc/4691/13170955"
 			(at 166.37 102.235 0)
 			(effects
@@
 	(symbol
 		(lib_id "entropy:COM-09426")
-		(at 118.11 83.82 0)
+		(at 116.84 83.82 0)
 		(unit 1)
 		(exclude_from_sim no)
@@
 		(fields_autoplaced yes)
 		(property "Reference" "U2"
-			(at 110.49 82.5499 0)
+			(at 109.22 82.5499 0)
 			(effects
 				(font
@@
 		)
 		(property "Value" "COM-09426"
-			(at 110.49 85.0899 0)
+			(at 109.22 85.0899 0)
 			(effects
 				(font
@@
 			)
 		)
-		(property "Footprint" ""
-			(at 115.57 83.82 0)
+		(property "Footprint" "entropy:COM-09426"
+			(at 114.3 83.82 0)
 			(effects
 				(font
@@
 		)
 		(property "Datasheet" ""
-			(at 115.57 83.82 0)
+			(at 114.3 83.82 0)
 			(effects
 				(font
@@
 		)
 		(property "Description" "https://www.sparkfun.com/products/9426"
-			(at 115.57 83.82 0)
-			(effects
-				(font
+			(at 114.3 83.82 0)
+			(effects
+				(font

Commit message: routing left keys pcb
Parts:
- SW44: footprint key-switches:SW_Gateron_LowProfile_HotSwap_THT -> key-switches:SW_Gateron_LowProfile_HotSwap_PTH
Changed lines of the file:
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@@
 			)
 		)
-		(property "Footprint" "key-switches:SW_Gateron_LowProfile_HotSwap_THT"
+		(property "Footprint" "key-switches:SW_Gateron_LowProfile_HotSwap_PTH"
 			(at 163.83 76.2 0)
 			(effects

Commit message: finished io board
Connections:
- net rclick_led_do: now reaches D87.1 (DO)
Changed lines of the file:
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@@
+	(wire
+		(pts
+			(xy 171.45 90.17) (xy 175.26 90.17)
+		)
+		(stroke
+			(width 0)
+			(type default)
+		)
+	)
 	(wire
 		(pts
@@
 			(effects
 				(font
+					(size 1.27 1.27)
+				)
+				(justify left)
+				(hide yes)
+			)
+		)
+	)
+	(global_label "rclick_led_do"
+		(shape input)
+		(at 175.26 90.17 0)
+		(fields_autoplaced yes)
+		(effects
+			(font
+				(size 1.27 1.27)
+			)
+			(justify left)
+		)
+		(property "Intersheetrefs" "${INTERSHEET_REFS}"
+			(at 190.6427 90.17 0)
+			(effects
+				(font
