File: corneds_devkit/io_board/right_ctrl.kicad_sch (KiCad schematic)
At the start: 0 parts

Commit message: added switch footprint, io sch, and keypad IC footprint. Need to find new LEDs and make joystick footprint
Parts:
- added R2: 10k, Resistor_SMD:R_0402_1005Metric, symbol Device:R
- added U4: ~, Package_DFN_QFN:WQFN-24-1EP_4x4mm_P0.5mm_EP2.45x2.45mm, symbol entropy:TCA8418
Connections:
- new net: R2.2, U4.15 (COL6), U4.16 (COL7), U4.17 (COL8), U4.18 (COL9), U4.5 (ROW3), U4.6 (ROW2), U4.7 (ROW1), U4.8 (ROW0)
- new net COL0R: U4.9 (COL0)
- new net COL1R: U4.10 (COL1)
- new net COL2R: U4.11 (COL2)
- new net COL3R: U4.12 (COL3)
- new net COL4R: U4.13 (COL4)
- new net COL5R: U4.14 (COL5)
- new net GNDR: U4.19 (GND)
- new net ROW0R: U4.1 (ROW7)
- new net ROW1R: U4.2 (ROW6)
- new net ROW2R: U4.3 (ROW5)
- new net ROW3R: U4.4 (ROW4)
- new net SCLR: U4.23 (SCL)
- new net SDAR: U4.22 (SDA)
- new net VDD_3V3R: R2.1, U4.21 (VCC)
- new net nINTR: U4.24 (nINT)
- new net nRESET: U4.20 (nRESET)

Commit message: finished routing power board and started on control board schematic but realized I need seperate reset lines
Parts:
- added R11: 10k, Resistor_SMD:R_0402_1005Metric, symbol Device:R
Connections:
- net GNDR: now also R11.2
- net nINTR: now also R11.1
Changed lines of the file:
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@@
 	(paper "A4")
+	(junction
+		(at 194.31 86.36)
+		(diameter 0)
+		(color 0 0 0 0)
+	)
 	(junction
 		(at 129.54 116.84)
@@
 	)
 	(junction
+		(at 163.83 127)
+		(diameter 0)
+		(color 0 0 0 0)
+	)
+	(junction
 		(at 129.54 111.76)
 		(diameter 0)
@@
 	(wire
 		(pts
-			(xy 163.83 125.73) (xy 163.83 128.27)
+			(xy 163.83 125.73) (xy 163.83 127)
 		)
 		(stroke
@@
 	(wire
 		(pts
+			(xy 163.83 127) (xy 163.83 128.27)
+		)
+		(stroke
+			(width 0)
+			(type default)
+		)
+	)
+	(wire
+		(pts
 			(xy 144.78 76.2) (xy 148.59 76.2)
 		)
@@
 	(wire
 		(pts
+			(xy 194.31 93.98) (xy 194.31 127)
+		)
+		(stroke
+			(width 0)
+			(type default)
+		)
+	)
+	(wire
+		(pts
 			(xy 148.59 91.44) (xy 129.54 91.44)
 		)
@@
 	(wire
 		(pts
+			(xy 194.31 127) (xy 163.83 127)
+		)
+		(stroke
+			(width 0)
+			(type default)
+		)
+	)
+	(wire
+		(pts
 			(xy 129.54 114.3) (xy 129.54 111.76)
 		)
@@
 	(wire
 		(pts
+			(xy 194.31 86.36) (xy 199.39 86.36)
+		)
+		(stroke
+			(width 0)
+			(type default)
+		)
+	)
+	(wire
+		(pts
 			(xy 144.78 109.22) (xy 148.59 109.22)
 		)
@@
 	(wire
 		(pts
-			(xy 179.07 86.36) (xy 182.88 86.36)
+			(xy 179.07 86.36) (xy 194.31 86.36)
 		)
 		(stroke
@@
 	(global_label "nINTR"
 		(shape input)
-		(at 182.88 86.36 0)
+		(at 199.39 86.36 0)
 		(fields_autoplaced yes)
 		(effects
@@
 		)
 		(property "Intersheetrefs" "${INTERSHEET_REFS}"
-			(at 191.1871 86.36 0)
+			(at 207.6971 86.36 0)
 			(effects
 				(font
@@
 					(unit 1)
 				)
+			)
+		)
+	)
+	(symbol
+		(lib_id "Device:R")
+		(at 194.31 90.17 0)
+		(unit 1)
+		(exclude_from_sim no)
+		(in_bom yes)
+		(on_board yes)
+		(dnp no)
+		(fields_autoplaced yes)
+		(property "Reference" "R11"
+			(at 196.85 88.8999 0)
+			(effects
+				(font
+					(size 1.27 1.27)
+				)
+				(justify left)
+			)
+		)
+		(property "Value" "10k"
+			(at 196.85 91.4399 0)
+			(effects
+				(font
+					(size 1.27 1.27)
+				)
+				(justify left)
+			)
+		)
+		(property "Footprint" "Resistor_SMD:R_0402_1005Metric"
+			(at 192.532 90.17 90)
+			(effects
+				(font
+					(size 1.27 1.27)
+				)
+				(hide yes)
+			)
+		)
+		(property "Datasheet" "~"
+			(at 194.31 90.17 0)
+			(effects
+				(font
+					(size 1.27 1.27)
+				)
+				(hide yes)
+			)
+		)
+		(property "Description" "Resistor"
+			(at 194.31 90.17 0)
+			(effects
+				(font
+					(size 1.27 1.27)
+				)
+				(hide yes)
+			)
+		)
+		(pin "1"
+		)
+		(pin "2"
+		)
+		(instances
+			(project "io_board"
+				(path "/244b6d6b-132d-4d50-ae86-e41103b29008/7cca1593-999d-4ccf-b76a-5f2d8940be69"
+					(reference "R11")
+					(unit 1)
+				)
