File: corneds_devkit/power_board/power_management.kicad_sch (KiCad schematic)
At the start: 26 parts, among them Q1 IRLML6401, Q2 IRLML6401, U1 AMS1117-3.3, U2 AMS1117-3.3, U3 MCP73831-2-OT, U4 MCP73831-2-OT

Commit message: ordered devkit rev A
Parts:
- removed C3: 10uF, Capacitor_SMD:C_01005_0402Metric, symbol Device:C_Polarized_US
- removed C4: 22uF, Capacitor_SMD:C_01005_0402Metric, symbol Device:C_Polarized_US
- removed C7: 4.7uF, Capacitor_SMD:C_0402_1005Metric, symbol Device:C
- removed C8: 4.7uF, symbol Device:C
- removed D2: 1N4148W, Diode_SMD:D_SOD-123, symbol Diode:1N4148W
- removed D4: LTST-C190KRKT, LED_SMD:LED_0201_0603Metric, symbol LED:CQY99
- removed Q2: IRLML6401, Package_TO_SOT_SMD:SOT-23, symbol Transistor_FET:IRLML6401
- removed R3, R4: 100kOhm, Resistor_SMD:R_01005_0402Metric, symbol Device:R_US
- removed R7: 2kOhm, Resistor_SMD:R_01005_0402Metric, symbol Device:R_US
- removed R8: 470Ohm, Resistor_SMD:R_01005_0402Metric, symbol Device:R_US
- removed U2: AMS1117-3.3, Package_TO_SOT_SMD:SOT-223-3_TabPin2, symbol Regulator_Linear:AMS1117-3.3
- removed U4: MCP73831-2-OT, Package_TO_SOT_SMD:SOT-23-5, symbol Battery_Management:MCP73831-2-OT
- C1: footprint Capacitor_SMD:C_01005_0402Metric -> Capacitor_SMD:C_0402_1005Metric
- C2: footprint Capacitor_SMD:C_01005_0402Metric -> Capacitor_SMD:C_0603_1608Metric
- C5: footprint (none) -> Capacitor_SMD:C_0402_1005Metric
- D3: footprint LED_SMD:LED_0201_0603Metric -> LED_SMD:LED_0603_1608Metric
- R1, R2, R5, R6: footprint Resistor_SMD:R_01005_0402Metric -> Resistor_SMD:R_0402_1005Metric
Connections:
- net 3_3VL renamed 3V3
- net BAT+L renamed BAT+
- net BAT_MEASL renamed BAT_MEAS
- net GNDL renamed GND
- net USB_5VL renamed USB_5V
Other:
- moved on the sheet: C1, C2, C5, C6, D1, D3, Q1, R1, R2, R5, R6, U1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
