File: corneds_devkit/power_board/power_board.kicad_pcb (KiCad board)
At the start: 2 copper layers, 44 x 34 mm, 19 parts, among them J1 BAT, Q1 IRLML6401, U1 AMS1117-3.3, U3 MCP73831-2-OT

Commit message: I'm assuming this is correcting the battery terminal
Parts:
- J2: moved to F.Cu
- turned J2 to 180 degrees
